File: Irrigation_System_PCB/Irrigation_System_PCB.kicad_pcb (KiCad board)
At the start: 2 copper layers, 4 parts, among them J1 Solenoid1, J2 baterie, U1 ESP32-S3-DevKitC

Commit message: f
Parts:
- added D2: D_Small, Diode_THT:D_A-405_P5.08mm_Vertical_AnodeUp, F.Cu at (314.6, 102.1)
- added D3: D_Small, Diode_THT:D_A-405_P5.08mm_Vertical_AnodeUp, F.Cu at (326.9, 81.7)
- added D4: D_Small, Diode_THT:D_A-405_P5.08mm_Vertical_AnodeUp, F.Cu at (338.4, 77.9)
- added D5: D_Small, Diode_THT:D_A-405_P5.08mm_Vertical_AnodeUp, F.Cu at (315.3, 93.6)
- added D6: D_Small, Diode_THT:D_A-405_P5.08mm_Vertical_AnodeUp, F.Cu at (326.9, 90.2)
- added D7: D_Small, Diode_THT:D_A-405_P5.08mm_Vertical_AnodeUp, F.Cu at (314.6, 97.9)
- added D8: D_Small, Diode_THT:D_A-405_P5.08mm_Vertical_AnodeUp, F.Cu at (183.9, 161.9)
- added D9: D_Small, Diode_THT:D_A-405_P5.08mm_Vertical_AnodeUp, F.Cu at (302.4, 109.7)
- added J10: 13.5-14V*_out, TerminalBlock:TerminalBlock_Altech_AK300-2_P5.00mm, F.Cu at (302.9, 72.6)
- added J11: Solenoid5*, TerminalBlock:TerminalBlock_Altech_AK300-2_P5.00mm, F.Cu at (279.8, 114.5)
- added J13: 12V*_in, TerminalBlock:TerminalBlock_Altech_AK300-2_P5.00mm, F.Cu at (279.8, 86.6)
- added J14: 5v_out, TerminalBlock:TerminalBlock_Altech_AK300-2_P5.00mm, F.Cu at (279.8, 100.5)
- added J4: Solenoid2, TerminalBlock:TerminalBlock_Altech_AK300-2_P5.00mm, F.Cu at (210.8, 150.6)
- added J5: Solenoid3, TerminalBlock:TerminalBlock_Altech_AK300-2_P5.00mm, F.Cu at (292.1, 86.6)
- added J6: adcon_input_wire, TerminalBlock:TerminalBlock_Altech_AK300-2_P5.00mm, F.Cu at (290.7, 72.6)
- added J7: Solenoid4, TerminalBlock:TerminalBlock_Altech_AK300-2_P5.00mm, F.Cu at (292.1, 100.5)
- added J8: Solenoid1, TerminalBlock:TerminalBlock_Altech_AK300-2_P5.00mm, F.Cu at (187.4, 150.9)
- added J9: 12V_in, TerminalBlock:TerminalBlock_Altech_AK300-2_P5.00mm, F.Cu at (278.4, 72.6)
- added K1: DIPxx-1Cxx-51x, Relay_THT:Relay_StandexMeder_DIP_LowProfile, F.Cu at (265.9, 68.7)
- added Q1: IRF3205, Package_TO_SOT_THT:TO-220-3_Vertical, F.Cu at (291.9, 117.4)
- added Q10: Q_NMOS_SGD, Package_TO_SOT_THT:TO-92L_Wide, F.Cu at (310.7, 109.5)
- added Q11: Q_NMOS_SGD, Package_TO_SOT_THT:TO-92L_Wide, F.Cu at (331.1, 97.0)
- added Q12: Q_NMOS_SGD, Package_TO_SOT_THT:TO-92L_Wide, F.Cu at (357.5, 69.6)
- added Q13: IRF3205, Package_TO_SOT_THT:TO-220-3_Vertical, F.Cu at (304.2, 97.5)
- added Q14: IRF3205, Package_TO_SOT_THT:TO-220-3_Vertical, F.Cu at (339.5, 69.5)
- added Q15: Q_NMOS_SGD, Package_TO_SOT_THT:TO-92L_Wide, F.Cu at (318.8, 108.3)
- added Q17: Q_NMOS_SGD, Package_TO_SOT_THT:TO-92L_Wide, F.Cu at (301.8, 120.1)
- added Q19: IRF3205, Package_TO_SOT_THT:TO-220-3_Vertical, F.Cu at (304.2, 103.4)
- added Q2: IRF3205, Package_TO_SOT_THT:TO-220-3_Vertical, F.Cu at (316.4, 89.4)
- added Q3: Q_NMOS_SGD, Package_TO_SOT_THT:TO-92L_Wide, F.Cu at (198.0, 172.8)
- added Q4: IRF3205, Package_TO_SOT_THT:TO-220-3_Vertical, F.Cu at (193.2, 161.8)
- added Q5: Q_NMOS_SGD, Package_TO_SOT_THT:TO-92L_Wide, F.Cu at (215.3, 173.5)
- added Q6: Q_NMOS_SGD, Package_TO_SOT_THT:TO-92L_Wide, F.Cu at (198.0, 166.3)
- added Q7: Q_NMOS_SGD, Package_TO_SOT_THT:TO-92L_Wide, F.Cu at (215.5, 166.5)
- added Q8: IRF3205, Package_TO_SOT_THT:TO-220-3_Vertical, F.Cu at (210.6, 162.1)
- added Q9: Q_NMOS_SGD, Package_TO_SOT_THT:TO-92L_Wide, F.Cu at (310.7, 116.0)
- added R1: 50k, Resistor_THT:R_Axial_DIN0204_L3.6mm_D1.6mm_P5.08mm_Vertical, F.Cu at (324.7, 10.2)
- added R10: DNP, Resistor_THT:R_Axial_DIN0204_L3.6mm_D1.6mm_P5.08mm_Vertical, F.Cu at (316.6, 7.01)
- added R11: 10k, Resistor_THT:R_Axial_DIN0204_L3.6mm_D1.6mm_P5.08mm_Vertical, F.Cu at (332.9, 22.8)
- added R12: 120, Resistor_THT:R_Axial_DIN0204_L3.6mm_D1.6mm_P5.08mm_Vertical, F.Cu at (349.1, 10.2)
- added R13: 10k, Resistor_THT:R_Axial_DIN0204_L3.6mm_D1.6mm_P5.08mm_Vertical, F.Cu at (184.1, 169.4)
- added R14: 10k, Resistor_THT:R_Axial_DIN0204_L3.6mm_D1.6mm_P5.08mm_Vertical, F.Cu at (349.1, 7.01)
- added R15: 10k, Resistor_THT:R_Axial_DIN0204_L3.6mm_D1.6mm_P5.08mm_Vertical, F.Cu at (184.0, 166.5)
- added R16: 10k, Resistor_THT:R_Axial_DIN0204_L3.6mm_D1.6mm_P5.08mm_Vertical, F.Cu at (316.6, 19.6)
- added R17: 10k, Resistor_THT:R_Axial_DIN0204_L3.6mm_D1.6mm_P5.08mm_Vertical, F.Cu at (332.9, 19.6)
- added R18: 10k, Resistor_THT:R_Axial_DIN0204_L3.6mm_D1.6mm_P5.08mm_Vertical, F.Cu at (324.7, 16.5)
- added R19: DNP, Resistor_THT:R_Axial_DIN0204_L3.6mm_D1.6mm_P5.08mm_Vertical, F.Cu at (341.0, 19.6)
- added R2: 10k, Resistor_THT:R_Axial_DIN0204_L3.6mm_D1.6mm_P5.08mm_Vertical, F.Cu at (316.6, 10.2)
- added R20: DNP, Resistor_THT:R_Axial_DIN0204_L3.6mm_D1.6mm_P5.08mm_Vertical, F.Cu at (316.6, 25.9)
- added R21: 10k, Resistor_THT:R_Axial_DIN0204_L3.6mm_D1.6mm_P5.08mm_Vertical, F.Cu at (324.7, 13.3)
- added R22: 10k, Resistor_THT:R_Axial_DIN0204_L3.6mm_D1.6mm_P5.08mm_Vertical, F.Cu at (332.9, 16.5)
- added R23: 10k, Resistor_THT:R_Axial_DIN0204_L3.6mm_D1.6mm_P5.08mm_Vertical, F.Cu at (341.0, 7.01)
- added R24: 10k, Resistor_THT:R_Axial_DIN0204_L3.6mm_D1.6mm_P5.08mm_Vertical, F.Cu at (332.9, 13.3)
- added R25: 10k, Resistor_THT:R_Axial_DIN0204_L3.6mm_D1.6mm_P5.08mm_Vertical, F.Cu at (341.0, 13.3)
- added R27: DNP, Resistor_THT:R_Axial_DIN0204_L3.6mm_D1.6mm_P5.08mm_Vertical, F.Cu at (332.9, 25.9)
- added R29: 10k, Resistor_THT:R_Axial_DIN0204_L3.6mm_D1.6mm_P5.08mm_Vertical, F.Cu at (324.7, 7.01)
- added R3: 10k, Resistor_THT:R_Axial_DIN0204_L3.6mm_D1.6mm_P5.08mm_Vertical, F.Cu at (324.7, 25.9)
- added R31: 10k, Resistor_THT:R_Axial_DIN0204_L3.6mm_D1.6mm_P5.08mm_Vertical, F.Cu at (324.7, 22.8)
- added R4: 10k, Resistor_THT:R_Axial_DIN0204_L3.6mm_D1.6mm_P5.08mm_Vertical, F.Cu at (316.6, 16.5)
- added R5: 5k, Resistor_THT:R_Axial_DIN0204_L3.6mm_D1.6mm_P5.08mm_Vertical, F.Cu at (316.6, 13.3)
- added R6: 10k, Resistor_THT:R_Axial_DIN0204_L3.6mm_D1.6mm_P5.08mm_Vertical, F.Cu at (332.9, 7.01)
- added R7: 10k, Resistor_THT:R_Axial_DIN0204_L3.6mm_D1.6mm_P5.08mm_Vertical, F.Cu at (193.1, 177.9)
- added R8: 10k, Resistor_THT:R_Axial_DIN0204_L3.6mm_D1.6mm_P5.08mm_Vertical, F.Cu at (324.7, 19.6)
- added R9: DNP, Resistor_THT:R_Axial_DIN0204_L3.6mm_D1.6mm_P5.08mm_Vertical, F.Cu at (189.1, 177.6)
- added SC1: Solar_Cells, TerminalBlock:TerminalBlock_Altech_AK300-2_P5.00mm, F.Cu at (327.4, 72.6)
- J1: value Solenoid1 -> 12V extern
- moved D1 211.3 mm to (302.4, 113.9)
- moved J1 180.3 mm to (267.6, 108.0)
Connections:
- J1 pad 1: +12V -> Net-(J1-Pad1)
- J1 pad 2: Net-(D1-Pad2) -> Net-(C4-Pad1)
- U1 pad 18: unconnected-(U1-Pad18) -> /ADC1
- U1 pad 21: unconnected-(U1-Pad21) -> +5V
