File: Irrigation_System_PCB/Irrigation_System_PCB.kicad_sch (KiCad schematic)
At the start: 13 parts, among them J1 Solenoid1, J2 baterie, U1 ESP32-S3-DevKitC

Commit message: Update Irrigation_System_PCB.kicad_sch
Parts:
- added C1, C2: C_Small, symbol Device:C_Small
- added D1, D3, D4, D5: D_Small, Diode_THT:D_A-405_P5.08mm_Vertical_AnodeUp, symbol Device:D_Small
- added J1: 12V extern, TerminalBlock:TerminalBlock_Altech_AK300-2_P5.00mm, symbol Connector:Screw_Terminal_01x02
- added J4: Solenoid4, TerminalBlock:TerminalBlock_Altech_AK300-2_P5.00mm, symbol Connector:Screw_Terminal_01x02
- added J5: Solenoid2, TerminalBlock:TerminalBlock_Altech_AK300-2_P5.00mm, symbol Connector:Screw_Terminal_01x02
- added J6: Solenoid3, TerminalBlock:TerminalBlock_Altech_AK300-2_P5.00mm, symbol Connector:Screw_Terminal_01x02
- added J?: Micro_SD_Card_Det, symbol Connector:Micro_SD_Card_Det
- added K1: DIPxx-1Cxx-51x, Relay_THT:Relay_StandexMeder_DIP_LowProfile, symbol Relay:DIPxx-1Cxx-51x
- added Q2, Q5, Q7: Q_PMOS_GSD, Package_TO_SOT_THT:TO-220-3_Horizontal_TabDown, symbol Device:Q_PMOS_GSD
- added Q4, Q6, Q8: Q_NMOS_SGD, Package_TO_SOT_THT:TO-92_Wide, symbol Device:Q_NMOS_SGD
- added R10, R13, R6: 10*, symbol Device:R_Small
- added R11, R12, R14, R4, R8, R9: 10k, symbol Device:R_Small
- added SC1: Solar_Cells, symbol Device:Solar_Cells
- gave numbers to parts that had none: 8
- renumbered D1 to D2, J1 to J3
Connections:
- net +12V: now also D1.1 (K), Q2.3 (D), Q5.3 (D), Q7.3 (D), R12.1, R4.1, R9.1
- net GND: now also D3.2 (A), D4.2 (A), D5.2 (A), J1.2 (Pin_2), J4.2 (Pin_2), J5.2 (Pin_2), J6.2 (Pin_2), K1.2, Q4.1 (S), Q6.1 (S), Q8.1 (S), R11.2, R14.2, R8.2, SC1.2 (-)
- net +5V: now reaches U1.21 (5V)
- net +12VA: no longer names the net of F1.2, J2.1 (Pin_1)
- new net: J1.1 (Pin_1), K1.14, K1.6
- new net: K1.1, SC1.1 (+)
- new net: K1.7, K1.8
- new net: Q8.2 (G), R13.2
- new net: Q6.2 (G), R10.2
- new net: Q4.2 (G), R6.2
- new net Valve2: R10.1, R11.1
- new net Valve3: R13.1, R14.1
- new net Valve4: R6.1, R8.1
- new net solenoid_gate2: Q5.1 (G), Q6.3 (D), R9.2
- new net solenoid_gate3: Q7.1 (G), Q8.3 (D), R12.2
- new net solenoid_gate4: Q2.1 (G), Q4.3 (D), R4.2
- new net solenoid_high2: D4.1 (K), J5.1 (Pin_1), Q5.2 (S)
- new net solenoid_high3: D5.1 (K), J6.1 (Pin_1), Q7.2 (S)
- new net solenoid_high4: D3.1 (K), J4.1 (Pin_1), Q2.2 (S)
Other:
- note added: "VALVA 1"
- note added: "VALVA 2"
- note added: "VALVA 3"
- note added: "VALVA 4"
- note added: "boost la 13-14V DC"
- note added: "buck 12-5 V"
- note added: "lef pe fiecare valva pt a vedea cand e pornita?"
- note added: "protectie polaritate inversa"
- moved on the sheet: D2, F1, J2, J3, Q1, Q3, R1, R2, R3, R5, R7

Commit message: g
Parts:
- removed D2, D3, D4, D5: D_Small, Diode_THT:D_A-405_P5.08mm_Vertical_AnodeUp, symbol Device:D_Small
- removed J3: Solenoid1, TerminalBlock:TerminalBlock_Altech_AK300-2_P5.00mm, symbol Connector:Screw_Terminal_01x02
- removed J4: Solenoid4, TerminalBlock:TerminalBlock_Altech_AK300-2_P5.00mm, symbol Connector:Screw_Terminal_01x02
- removed J5: Solenoid2, TerminalBlock:TerminalBlock_Altech_AK300-2_P5.00mm, symbol Connector:Screw_Terminal_01x02
- removed J6: Solenoid3, TerminalBlock:TerminalBlock_Altech_AK300-2_P5.00mm, symbol Connector:Screw_Terminal_01x02
- removed Q1, Q2, Q5, Q7: Q_PMOS_GSD, Package_TO_SOT_THT:TO-220-3_Horizontal_TabDown, symbol Device:Q_PMOS_GSD
- removed Q3, Q4, Q6, Q8: Q_NMOS_SGD, Package_TO_SOT_THT:TO-92_Wide, symbol Device:Q_NMOS_SGD
- removed R10, R13, R5, R6: 10*, symbol Device:R_Small
- removed R11, R12, R14, R3, R4, R7, R8, R9: 10k, symbol Device:R_Small
- added C?: C_Small, symbol Device:C_Small
- added C? (x2): 100n, symbol Device:C_Small
- added D? (x5): D_Small, Diode_THT:D_A-405_P5.08mm_Vertical_AnodeUp, symbol Device:D_Small
- added J? (x4): Solenoid1, TerminalBlock:TerminalBlock_Altech_AK300-2_P5.00mm, symbol Connector:Screw_Terminal_01x02
- added Q? (x4): Q_PNP_CBE, Package_TO_SOT_THT:TO-92L_Wide, symbol Device:Q_PNP_CBE
- added Q? (x2): IRF3205, Package_TO_SOT_THT:TO-220-3_Vertical, symbol Transistor_FET:IRF3205
- added Q? (x4): IRF3205, Package_TO_SOT_THT:TO-220-3_Horizontal_TabDown, symbol Transistor_FET:IRF3205
- added R? (x4): 1k, symbol Device:R_Small
- added R? (x6): 10k, symbol Device:R_Small
Connections:
- net +12V: now also D?.1 (K), D?.1 (K), D?.1 (K), D?.1 (K), D?.1 (K), J?.1 (Pin_1), J?.1 (Pin_1), J?.1 (Pin_1), J?.1 (Pin_1), R?.1, R?.1, R?.1, R?.1
- net ADC1: now also C1.2
- net GND: now also C1.1, C2.2, D?.2 (A), Q?.3 (E), Q?.3 (E), Q?.3 (E), Q?.3 (E), Q?.3 (S), Q?.3 (S), Q?.3 (S), Q?.3 (S), Q?.3 (S), Q?.3 (S); no longer J1.2 (Pin_2), SC1.2 (-)
- net Valve1: now also R?.1, R?.1, R?.1, R?.1
- net at J1.1 (Pin_1), K1.14, K1.6: now also C?.1, R?.1
- net at K1.1, SC1.1 (+): now also C?.1, R?.1
- net at K1.7, K1.8: now also C2.1
- new net: J1.2 (Pin_2), Q?.2 (D)
- new net: D?.2 (A), J?.2 (Pin_2), Q?.2 (D) (x4)
- new net: C?.2, Q?.1 (G), R?.2 (x2)
- new net: Q?.2 (B), R?.2 (x4)
- new net: Q?.1 (C), Q?.1 (G), R?.2 (x4)
- new net: Q?.2 (D), SC1.2 (-)
Other:
- moved on the sheet: C1, J1, SC1

Commit message: Update Irrigation_System_PCB.kicad_sch
Parts:
- added C7, C8: C_Small, symbol Device:C_Small
- added D5, D6: D_Small, Diode_THT:D_A-405_P5.08mm_Vertical_AnodeUp, symbol Device:D_Small
- added J6: adcon_input_wire, TerminalBlock:TerminalBlock_Altech_AK300-2_P5.00mm, symbol Connector:Screw_Terminal_01x02
- added J?: 12V_in, TerminalBlock:TerminalBlock_Altech_AK300-2_P5.00mm, symbol Connector:Screw_Terminal_01x02
- added J?: Conn_01x04, symbol Connector_Generic:Conn_01x04
- added J?: 13.5-14V*_out, TerminalBlock:TerminalBlock_Altech_AK300-2_P5.00mm, symbol Connector:Screw_Terminal_01x02
- added J?: 5v_out, TerminalBlock:TerminalBlock_Altech_AK300-2_P5.00mm, symbol Connector:Screw_Terminal_01x02
- added J?: 12V*_in, TerminalBlock:TerminalBlock_Altech_AK300-2_P5.00mm, symbol Connector:Screw_Terminal_01x02
- added R11, R6: 10k, symbol Device:R_Small
- added R12: 120, symbol Device:R_Small
- added R5: 5k, symbol Device:R_Small
- added U2: AD8620, symbol Amplifier_Operational:AD8620
- R13, R14, R7, R8: renamed from R?; value 10k -> 1k
- gave numbers to parts that had none: 29
Connections:
- net +12V: now also C6.1, J?.1 (Pin_1)
- net +3V3: now also R5.1, U2.8 (V+)
- net +5V: now also J?.1 (Pin_1)
- net GND: now also C6.2, C8.2, D6.1 (K), J6.2 (Pin_2), J?.1 (Pin_1), J?.1 (Pin_1), J?.1 (Pin_1), J?.2 (Pin_2), J?.2 (Pin_2), R11.1, R6.2, U2.4 (V-)
- net at C4.1, K1.14, K1.6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: now also J1.2 (Pin_2); no longer J1.1 (Pin_1)
- net at Q1.2 (D): now also J1.1 (Pin_1); no longer J1.2 (Pin_2)
- net at C2.1, K1.7, K1.8: now also J?.2 (Pin_2)
- net at D1.2 (A): now also J?.2 (Pin_2)
- new net: C7.2, D5.1 (K), D6.2 (A)
- new net: C8.1, D5.2 (A), R12.2
- new net: R5.2, R6.1, U2.2 (-)
- new net: J6.1 (Pin_1), U2.3 (+), U2.5 (+)
- new net: R11.2, R12.1, U2.6 (-)
- new net I2C_ext_CLK: J?.2 (Pin_2)
- new net I2C_ext_SDA: J?.3 (Pin_3)
- new net PWM_pin: C7.1
- new net adcon+: U2.1
- new net adcon-: U2.7
- no-connect marks 0 -> 1
Other:
- note added: "+ side vith 2V offset"
- note added: "- side with -2V offset"
- note added: "Adcon trimite: pulsuri de +5-15V pt a porni valva pulsuri de -5-15V pt a opri valva"
- note added: "charge pump"
- moved on the sheet: C1, C6, D1, D2, F1, J1, J2, R1, R2

Commit message: f
Parts:
- removed Q10, Q5, Q6, Q9: Q_PNP_CBE, Package_TO_SOT_THT:TO-92L_Wide, symbol Device:Q_PNP_CBE
- removed Q3, Q7: IRF3205, Package_TO_SOT_THT:TO-220-3_Horizontal_TabDown, symbol Transistor_FET:IRF3205
- added D9: D_Small, Diode_THT:D_A-405_P5.08mm_Vertical_AnodeUp, symbol Device:D_Small
- added J11: Solenoid5*, TerminalBlock:TerminalBlock_Altech_AK300-2_P5.00mm, symbol Connector:Screw_Terminal_01x02
- added Q10, Q11, Q12, Q15, Q17, Q3, Q5, Q6, Q7, Q9: Q_NMOS_SGD, Package_TO_SOT_THT:TO-92L_Wide, symbol Device:Q_NMOS_SGD
- added Q13, Q14, Q19: IRF3205, Package_TO_SOT_THT:TO-220-3_Vertical, symbol Transistor_FET:IRF3205
- added R17, R18, R21, R22, R23, R24, R25, R29, R31: 10k, Resistor_THT:R_Axial_DIN0204_L3.6mm_D1.6mm_P5.08mm_Vertical, symbol Device:R_Small
- added R19, R20, R27: DNP, Resistor_THT:R_Axial_DIN0204_L3.6mm_D1.6mm_P5.08mm_Vertical, symbol Device:R_Small
- J4: value Solenoid1 -> Solenoid2
- J5: value Solenoid1 -> Solenoid3
- J7: value Solenoid1 -> Solenoid4
- Q4, Q8: footprint Package_TO_SOT_THT:TO-220-3_Horizontal_TabDown -> Package_TO_SOT_THT:TO-220-3_Vertical
- R1, R11, R12, R2, R3, R4, R5, R6: footprint (none) -> Resistor_THT:R_Axial_DIN0204_L3.6mm_D1.6mm_P5.08mm_Vertical
- R10, R9: value 1k -> DNP; footprint (none) -> Resistor_THT:R_Axial_DIN0204_L3.6mm_D1.6mm_P5.08mm_Vertical; notes (none) -> -short for PNP
- R13, R14, R15, R16, R7, R8: value 1k -> 10k; footprint (none) -> Resistor_THT:R_Axial_DIN0204_L3.6mm_D1.6mm_P5.08mm_Vertical
- SC1: footprint (none) -> TerminalBlock:TerminalBlock_Altech_AK300-2_P5.00mm
- gave numbers to parts that had none: 5
Connections:
- net +12V: now also R15.1, R16.1, D9.1 (K), J11.1 (Pin_1), R23.1, R24.1, R31.1; no longer R13.1, R14.1, R7.1, R8.1
- net +3V3: now also R13.1, R14.1, R21.1, R22.1, R29.1
- net GND: now also R7.2, R8.2, Q10.1 (S), Q11.1 (S), Q12.1 (S), Q13.3 (S), Q14.3 (S), Q15.1 (S), Q17.1 (S), Q19.3 (S), Q3.1 (S), Q5.1 (S), Q6.1 (S), Q7.1 (S), Q9.1 (S), R17.2, R18.2, R25.2
- net at D3.2 (A), J4.2 (Pin_2): now also Q8.2 (D)
- net at D4.2 (A), J5.2 (Pin_2): now also Q13.2 (D); no longer Q4.2 (D)
- net at R9.2: now also R13.2, Q3.3 (D), Q6.2 (G)
- net at R15.2: now also Q4.1 (G), Q6.3 (D)
- net at D8.2 (A), J8.2 (Pin_2): now also Q4.2 (D); no longer Q8.2 (D)
- net at D7.2 (A), J7.2 (Pin_2): now also Q14.2 (D)
- net at R10.2: now also R14.2, Q5.3 (D), Q7.2 (G)
- net at Q8.1 (G): now also R16.2, Q7.3 (D); no longer R14.2
- removed net Valve1: R10.1, R15.1, R16.1, R9.1
- new net: Q15.3 (D), Q17.2 (G), R27.2, R29.2
- new net: Q11.2 (G), Q9.3 (D), R19.2, R21.2
- new net: Q17.3 (D), Q19.1 (G), R31.2
- new net: D9.2 (A), J11.2 (Pin_2), Q19.2 (D)
- new net: Q10.3 (D), Q12.2 (G), R20.2, R22.2
- new net: Q11.3 (D), Q13.1 (G), R23.2
- new net: Q12.3 (D), Q14.1 (G), R24.2
- new net VALVE1: Q3.2 (G), R7.1, R9.1
- new net VALVE3: Q9.2 (G), R17.1, R19.1
- new net VALVE4: Q10.2 (G), Q5.2 (G), R10.1, R18.1, R20.1, R8.1
- new net VALVE5: Q15.2 (G), R25.1, R27.1
Other:
- note removed: "VALVA 1"
- note removed: "VALVA 2"
- note removed: "VALVA 3"
- note removed: "VALVA 4"
- note removed: "lef pe fiecare valva pt a vedea cand e pornita?"
- moved on the sheet: C7, C8, D5, D6, D8, J15, J6, J8, Q4, R11, R12, R5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
